File: V1/eumesmo-rl-8ch8a-v1.kicad_pcb (KiCad board)
At the start: 2 copper layers, 98 x 67.8 mm, 48 parts, among them J1 250-202, J2 250-204, J3 250-204, J4 DB142V-5.08-4P, J5 DB142V-5.08-4P, J6 DB142V-5.08-4P, J7 DB142V-5.08-4P, K1 G5Q-1A4-DC24V, K2 G5Q-1A4-DC24V, K3 G5Q-1A4-DC24V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

Commit message: Release V1.2.0
Other:
- board text added: "V1.2 2026-06-17"
- board text removed: "V1.2 2026-06-13"
Changed lines of the file:
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@@
 	(title_block
 		(title "eumesmo 8x 24V 8A NO Relay Module")
-		(date "2026-06-13")
+		(date "2026-06-17")
 		(rev "V1.2")
 	)
@@
 		(layer "F.SilkS")
 	)
+	(gr_rect
+		(start 128.5 77.5)
+		(end 136 79)
+		(stroke
+			(width 0.1)
+			(type solid)
+		)
+		(fill no)
+		(layer "F.SilkS")
+	)
 	(gr_line
 		(start 131.58 124.5)
@@
 		(layer "F.SilkS")
 	)
-	(gr_rect
-		(start 151.5 74.75)
-		(end 157 77.5)
-		(stroke
-			(width 0.1)
-			(type solid)
-		)
-		(fill no)
-		(layer "F.SilkS")
-	)
 	(gr_line
 		(start 155.48 124.5)
@@
 		(layer "Edge.Cuts")
 	)
-	(gr_text "V1.2\n2026-06-13"
-		(at 154.25 76 0)
+	(gr_text "V1.2 2026-06-17"
+		(at 132.25 78.25 0)
 		(layer "F.SilkS")
 		(effects
