File: V1/eumesmo-rl-8ch8a-v1.kicad_pcb (KiCad board)
At the start: 2 copper layers, 98 x 67.8 mm, 48 parts, among them J1 250-202, J2 250-204, J3 250-204, J4 DB142V-5.08-4P, J5 DB142V-5.08-4P, J6 DB142V-5.08-4P, J7 DB142V-5.08-4P, K1 G5Q-1A4-DC24V, K2 G5Q-1A4-DC24V, K3 G5Q-1A4-DC24V, K4 G5Q-1A4-DC24V, K5 G5Q-1A4-DC24V, K6 G5Q-1A4-DC24V, K7 G5Q-1A4-DC24V, K8 G5Q-1A4-DC24V

Commit message: Replaced 0603 size 10k resistor for 0805 size.
Parts:
- R1, R2, R3, R4, R5, R6, R7, R8: value 10k/100mW -> 10k/125mW; footprint Tales:R_0603_1608Metric -> Tales:R_0805_2012Metric
- moved R5 1.52 mm to (194.2, 64.8)
- moved R1 1.50 mm to (150.2, 67.0)
- moved R6 1.03 mm to (194.2, 66.8)
- moved R2 1.00 mm to (150.2, 69.0)
- moved R7 0.56 mm to (194.2, 68.8)
- moved R3 0.50 mm to (150.2, 71.0)
- moved R8 0.25 mm to (194.2, 70.8)
Routing:
- net +24V: track 232.6 -> 220.4 mm, vias 0 -> 2
- net /LED5: track 22.4 -> 19.7 mm
- net /LED6: track 15.7 -> 13.9 mm
- net /LED7: track 9.24 -> 8.06 mm
- net /LED1: track 20.3 -> 20.8 mm
