File: V1/eumesmo-rl-8ch8a-v1.kicad_pcb (KiCad board)
At the start: 2 copper layers, 98 x 67.8 mm, 48 parts, among them J1 250-202, J2 250-204, J3 250-204, J4 DB142V-5.08-4P, J5 DB142V-5.08-4P, J6 DB142V-5.08-4P, J7 DB142V-5.08-4P, K1 G5Q-1A4-DC24V, K2 G5Q-1A4-DC24V, K3 G5Q-1A4-DC24V, K4 G5Q-1A4-DC24V, K5 G5Q-1A4-DC24V, K6 G5Q-1A4-DC24V, K7 G5Q-1A4-DC24V, K8 G5Q-1A4-DC24V

Commit message: Revised Metaltex holders
Other:
- board text added: "SUPORTES PCI METALTEX SP7 1x pé macho 9 mm 1x pé fêmea 9 mm 1x espaçador 45 mm 1x espaçador 20 mm 1x espaçador 15 mm Comprimento total 98 mm Largura da placa 67,8 mm"
- board text removed: "SUPORTES PCI METALTEX SP7 1x pé macho 9 mm 1x pé fêmea 9 mm 1x espaçador 30 mm 1x espaçador 10 mm Comprimento total 58 mm Largura da placa 67,8 mm"
Changed lines of the file:
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@@
 		)
 	)
-	(gr_text "SUPORTES PCI METALTEX SP7\n1x pé macho  9 mm\n1x pé fêmea 9 mm\n1x espaçador 30 mm\n1x espaçador 10 mm\nComprimento total 58 mm\nLargura da placa 67,8 mm"
+	(gr_text "SUPORTES PCI METALTEX SP7\n1x pé macho  9 mm\n1x pé fêmea 9 mm\n1x espaçador 45 mm\n1x espaçador 20 mm\n1x espaçador 15 mm\nComprimento total 98 mm\nLargura da placa 67,8 mm"
 		(at 125 132 0)
 		(layer "Cmts.User")
