File: V1/eumesmo-rl-8ch8a-v1.kicad_sch (KiCad schematic)
At the start: 47 parts, among them J1 250-202, J2 250-204, J3 250-204, J4 DB142V-5.08-4P, J5 DB142V-5.08-4P, J6 DB142V-5.08-4P, J7 DB142V-5.08-4P, K1 G5Q-1A4-DC24V, K2 G5Q-1A4-DC24V, K3 G5Q-1A4-DC24V, K4 G5Q-1A4-DC24V, K5 G5Q-1A4-DC24V, K6 G5Q-1A4-DC24V, K7 G5Q-1A4-DC24V, K8 G5Q-1A4-DC24V

Commit message: Replaced 0603 size 10k resistor for 0805 size.
Parts:
- R1, R2, R3, R4, R5, R6, R7, R8: value 10k/100mW -> 10k/125mW; footprint Tales:R_0603_1608Metric -> Tales:R_0805_2012Metric; LCSC Part # C25804 -> C17414; Mfr UNI-ROYAL(Uniroyal Elec) -> Uniroyal; Mfr PN 0603WAF1002T5E -> 0805W8F1002T5E; Package 0603/1608 -> 0805/2012; Vendor PN C25804 -> C17414
Changed lines of the file:
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@@
 			)
 		)
-		(property "Value" "10k/100mW"
+		(property "Value" "10k/125mW"
 			(at 170.18 110.49 0)
 			(show_name no)
@@
 			)
 		)
-		(property "Footprint" "Tales:R_0603_1608Metric"
+		(property "Footprint" "Tales:R_0805_2012Metric"
 			(at 173.736 110.744 90)
 			(hide yes)
@@
 			)
 		)
-		(property "Mfr" "UNI-ROYAL(Uniroyal Elec)"
+		(property "Mfr" "Uniroyal"
 			(at 172.72 110.49 0)
 			(hide yes)
@@
 			)
 		)
-		(property "Mfr PN" "0603WAF1002T5E"
+		(property "Mfr PN" "0805W8F1002T5E"
 			(at 172.72 110.49 0)
 			(hide yes)
@@
 			)
 		)
-		(property "Vendor PN" "C25804"
+		(property "Vendor PN" "C17414"
 			(at 172.72 110.49 0)
 			(hide yes)
@@
 			)
 		)
-		(property "LCSC Part #" "C25804"
+		(property "LCSC Part #" "C17414"
 			(at 170.18 113.03 0)
 			(show_name no)
@@
 			)
 		)
-		(property "Package" "0603/1608"
+		(property "Package" "0805/2012"
 			(at 172.72 110.49 0)
 			(hide yes)
@@
 			)
 		)
-		(property "Value" "10k/100mW"
+		(property "Value" "10k/125mW"
 			(at 170.18 148.59 0)
 			(show_name no)
@@
 			)
 		)
-		(property "Footprint" "Tales:R_0603_1608Metric"
+		(property "Footprint" "Tales:R_0805_2012Metric"
 			(at 173.736 148.844 90)
 			(hide yes)
@@
 			)
 		)
-		(property "Mfr" "UNI-ROYAL(Uniroyal Elec)"
+		(property "Mfr" "Uniroyal"
 			(at 172.72 148.59 0)
 			(hide yes)
@@
 			)
 		)
-		(property "Mfr PN" "0603WAF1002T5E"
+		(property "Mfr PN" "0805W8F1002T5E"
 			(at 172.72 148.59 0)
 			(hide yes)
@@
 			)
 		)
-		(property "Vendor PN" "C25804"
+		(property "Vendor PN" "C17414"
 			(at 172.72 148.59 0)
 			(hide yes)
@@
 			)
 		)
-		(property "LCSC Part #" "C25804"
+		(property "LCSC Part #" "C17414"
 			(at 170.18 151.13 0)
 			(show_name no)
@@
 			)
 		)
-		(property "Package" "0603/1608"
+		(property "Package" "0805/2012"
 			(at 172.72 148.59 0)
 			(hide yes)
@@
 			)
 		)
-		(property "Value" "10k/100mW"
+		(property "Value" "10k/125mW"
 			(at 73.66 31.75 0)
 			(show_name no)
@@
 			)
 		)
-		(property "Footprint" "Tales:R_0603_1608Metric"
+		(property "Footprint" "Tales:R_0805_2012Metric"
 			(at 77.216 32.004 90)
 			(hide yes)
@@
 			)
 		)
-		(property "Mfr" "UNI-ROYAL(Uniroyal Elec)"
+		(property "Mfr" "Uniroyal"
 			(at 76.2 31.75 0)
 			(hide yes)
@@
 			)
 		)
-		(property "Mfr PN" "0603WAF1002T5E"
+		(property "Mfr PN" "0805W8F1002T5E"
 			(at 76.2 31.75 0)
 			(hide yes)
@@
 			)
 		)
-		(property "Vendor PN" "C25804"
+		(property "Vendor PN" "C17414"
 			(at 76.2 31.75 0)
 			(hide yes)
@@
 			)
 		)
-		(property "LCSC Part #" "C25804"
+		(property "LCSC Part #" "C17414"
 			(at 73.66 34.29 0)
 			(show_name no)
@@
 			)
 		)
-		(property "Package" "0603/1608"
+		(property "Package" "0805/2012"
 			(at 76.2 31.75 0)
 			(hide yes)
@@
 			)
 		)
-		(property "Value" "10k/100mW"
+		(property "Value" "10k/125mW"
 			(at 73.66 107.95 0)
 			(show_name no)
@@
 			)
 		)
-		(property "Footprint" "Tales:R_0603_1608Metric"
+		(property "Footprint" "Tales:R_0805_2012Metric"
 			(at 77.216 108.204 90)
 			(hide yes)
@@
 			)
 		)
-		(property "Mfr" "UNI-ROYAL(Uniroyal Elec)"
+		(property "Mfr" "Uniroyal"
 			(at 76.2 107.95 0)
 			(hide yes)
@@
 			)
 		)
-		(property "Mfr PN" "0603WAF1002T5E"
+		(property "Mfr PN" "0805W8F1002T5E"
 			(at 76.2 107.95 0)
 			(hide yes)
@@
 			)
 		)
-		(property "Vendor PN" "C25804"
+		(property "Vendor PN" "C17414"
 			(at 76.2 107.95 0)
 			(hide yes)
@@
 			)
 		)
-		(property "LCSC Part #" "C25804"
+		(property "LCSC Part #" "C17414"
 			(at 73.66 110.49 0)
 			(show_name no)
@@
 			)
 		)
-		(property "Package" "0603/1608"
+		(property "Package" "0805/2012"
 			(at 76.2 107.95 0)
 			(hide yes)
@@
 			)
 		)
-		(property "Value" "10k/100mW"
+		(property "Value" "10k/125mW"
 			(at 73.66 69.85 0)
 			(show_name no)
@@
 			)
 		)
-		(property "Footprint" "Tales:R_0603_1608Metric"
+		(property "Footprint" "Tales:R_0805_2012Metric"
 			(at 77.216 70.104 90)
 			(hide yes)
@@
 			)
 		)
-		(property "Mfr" "UNI-ROYAL(Uniroyal Elec)"
+		(property "Mfr" "Uniroyal"
 			(at 76.2 69.85 0)
 			(hide yes)
@@
 			)
 		)
-		(property "Mfr PN" "0603WAF1002T5E"
+		(property "Mfr PN" "0805W8F1002T5E"
 			(at 76.2 69.85 0)
 			(hide yes)
@@
 			)
 		)
-		(property "Vendor PN" "C25804"
+		(property "Vendor PN" "C17414"
 			(at 76.2 69.85 0)
 			(hide yes)
@@
 			)
 		)
-		(property "LCSC Part #" "C25804"
+		(property "LCSC Part #" "C17414"
 			(at 73.66 72.39 0)
 			(show_name no)
@@
 			)
 		)
-		(property "Package" "0603/1608"
+		(property "Package" "0805/2012"
 			(at 76.2 69.85 0)
 			(hide yes)
@@
 			)
 		)
-		(property "Value" "10k/100mW"
+		(property "Value" "10k/125mW"
 			(at 170.18 72.39 0)
 			(show_name no)
@@
 			)
 		)
-		(property "Footprint" "Tales:R_0603_1608Metric"
+		(property "Footprint" "Tales:R_0805_2012Metric"
 			(at 173.736 72.644 90)
 			(hide yes)
@@
 			)
 		)
-		(property "Mfr" "UNI-ROYAL(Uniroyal Elec)"
+		(property "Mfr" "Uniroyal"
 			(at 172.72 72.39 0)
 			(hide yes)
@@
 			)
 		)
-		(property "Mfr PN" "0603WAF1002T5E"
+		(property "Mfr PN" "0805W8F1002T5E"
 			(at 172.72 72.39 0)
 			(hide yes)
@@
 			)
 		)
-		(property "Vendor PN" "C25804"
+		(property "Vendor PN" "C17414"
 			(at 172.72 72.39 0)
 			(hide yes)
@@
 			)
 		)
-		(property "LCSC Part #" "C25804"
+		(property "LCSC Part #" "C17414"
 			(at 170.18 74.93 0)
 			(show_name no)
@@
 			)
 		)
-		(property "Package" "0603/1608"
+		(property "Package" "0805/2012"
 			(at 172.72 72.39 0)
 			(hide yes)
@@
 			)
 		)
-		(property "Value" "10k/100mW"
+		(property "Value" "10k/125mW"
 			(at 73.66 146.05 0)
 			(show_name no)
@@
 			)
 		)
-		(property "Footprint" "Tales:R_0603_1608Metric"
+		(property "Footprint" "Tales:R_0805_2012Metric"
 			(at 77.216 146.304 90)
 			(hide yes)
@@
 			)
 		)
-		(property "Mfr" "UNI-ROYAL(Uniroyal Elec)"
+		(property "Mfr" "Uniroyal"
 			(at 76.2 146.05 0)
 			(hide yes)
@@
 			)
 		)
-		(property "Mfr PN" "0603WAF1002T5E"
+		(property "Mfr PN" "0805W8F1002T5E"
 			(at 76.2 146.05 0)
 			(hide yes)
@@
 			)
 		)
-		(property "Vendor PN" "C25804"
+		(property "Vendor PN" "C17414"
 			(at 76.2 146.05 0)
 			(hide yes)
@@
 			)
 		)
-		(property "LCSC Part #" "C25804"
+		(property "LCSC Part #" "C17414"
 			(at 73.66 148.59 0)
 			(show_name no)
@@
 			)
 		)
-		(property "Package" "0603/1608"
+		(property "Package" "0805/2012"
 			(at 76.2 146.05 0)
 			(hide yes)
@@
 			)
 		)
-		(property "Value" "10k/100mW"
+		(property "Value" "10k/125mW"
 			(at 170.18 34.29 0)
 			(show_name no)
@@
 			)
 		)
-		(property "Footprint" "Tales:R_0603_1608Metric"
+		(property "Footprint" "Tales:R_0805_2012Metric"
 			(at 173.736 34.544 90)
 			(hide yes)
@@
 			)
 		)
-		(property "Mfr" "UNI-ROYAL(Uniroyal Elec)"
+		(property "Mfr" "Uniroyal"
 			(at 172.72 34.29 0)
 			(hide yes)
@@
 			)
 		)
-		(property "Mfr PN" "0603WAF1002T5E"
+		(property "Mfr PN" "0805W8F1002T5E"
 			(at 172.72 34.29 0)
 			(hide yes)
@@
 			)
 		)
-		(property "Vendor PN" "C25804"
+		(property "Vendor PN" "C17414"
 			(at 172.72 34.29 0)
 			(hide yes)
@@
 			)
 		)
-		(property "LCSC Part #" "C25804"
+		(property "LCSC Part #" "C17414"
 			(at 170.18 36.83 0)
 			(show_name no)
@@
 			)
 		)
-		(property "Package" "0603/1608"
+		(property "Package" "0805/2012"
 			(at 172.72 34.29 0)
 			(hide yes)

Commit message: LEDs changed to orange
Parts:
- D1, D11, D13, D15, D3, D5, D7, D9: value EMERALD -> ORANGE/0603; LCSC Part # C2984266 -> C2987557; Mfr PN 19-213/GHC-XS1T1N/5T -> 19-217/S2C-AL1M2VY/6T; Vendor PN C2984266 -> C2987557
- R1, R2, R3, R4, R5, R6, R7, R8: value 10k/125mW -> 9.1k/125mW; LCSC Part # C17414 -> C17855; Mfr PN 0805W8F1002T5E -> 0805W8F9101T5E; Vendor PN C17414 -> C17855
Other:
- note added: "V_{F} = 1,8V @ 2,5mA I_{LED} = (24V - V_{F}) / R I_{LED} = (24V - 1.8V) / 9.1k I_{LED} = 2.44 mA"
Changed lines of the file:
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@@
 		(rev "V1.2")
 	)
+	(text "V_{F} = 1,8V @ 2,5mA\nI_{LED} = (24V - V_{F}) / R\nI_{LED} = (24V - 1.8V) / 9.1k\nI_{LED} = 2.44 mA"
+		(exclude_from_sim no)
+		(at 66.04 179.07 0)
+		(effects
+			(font
+				(size 1.5 1.5)
+			)
+			(justify left bottom)
+		)
+	)
 	(junction
 		(at 181.61 163.83)
@@
 			)
 		)
-		(property "Value" "EMERALD"
+		(property "Value" "ORANGE/0603"
 			(at 73.66 156.21 90)
 			(show_name no)
@@
 			)
 		)
-		(property "Mfr PN" "19-213/GHC-XS1T1N/5T"
+		(property "Mfr PN" "19-217/S2C-AL1M2VY/6T"
 			(at 76.2 156.21 0)
 			(hide yes)
@@
 			)
 		)
-		(property "Vendor PN" "C2984266"
+		(property "Vendor PN" "C2987557"
 			(at 76.2 156.21 0)
 			(hide yes)
@@
 			)
 		)
-		(property "LCSC Part #" "C2984266"
+		(property "LCSC Part #" "C2987557"
 			(at 73.66 158.75 90)
 			(show_name no)
@@
 			)
 		)
-		(property "Value" "EMERALD"
+		(property "Value" "ORANGE/0603"
 			(at 170.18 82.55 90)
 			(show_name no)
@@
 			)
 		)
-		(property "Mfr PN" "19-213/GHC-XS1T1N/5T"
+		(property "Mfr PN" "19-217/S2C-AL1M2VY/6T"
 			(at 172.72 82.55 0)
 			(hide yes)
@@
 			)
 		)
-		(property "Vendor PN" "C2984266"
+		(property "Vendor PN" "C2987557"
 			(at 172.72 82.55 0)
 			(hide yes)
@@
 			)
 		)
-		(property "LCSC Part #" "C2984266"
+		(property "LCSC Part #" "C2987557"
 			(at 170.18 85.09 90)
 			(show_name no)
@@
 			)
 		)
-		(property "Value" "10k/125mW"
+		(property "Value" "9.1k/125mW"
 			(at 170.18 110.49 0)
 			(show_name no)
@@
 			)
 		)
-		(property "Mfr PN" "0805W8F1002T5E"
+		(property "Mfr PN" "0805W8F9101T5E"
 			(at 172.72 110.49 0)
 			(hide yes)
@@
 			)
 		)
-		(property "Vendor PN" "C17414"
+		(property "Vendor PN" "C17855"
 			(at 172.72 110.49 0)
 			(hide yes)
@@
 			)
 		)
-		(property "LCSC Part #" "C17414"
+		(property "LCSC Part #" "C17855"
 			(at 170.18 113.03 0)
 			(show_name no)
@@
 			)
 		)
-		(property "Value" "10k/125mW"
+		(property "Value" "9.1k/125mW"
 			(at 170.18 148.59 0)
 			(show_name no)
@@
 			)
 		)
-		(property "Mfr PN" "0805W8F1002T5E"
+		(property "Mfr PN" "0805W8F9101T5E"
 			(at 172.72 148.59 0)
 			(hide yes)
@@
 			)
 		)
-		(property "Vendor PN" "C17414"
+		(property "Vendor PN" "C17855"
 			(at 172.72 148.59 0)
 			(hide yes)
@@
 			)
 		)
-		(property "LCSC Part #" "C17414"
+		(property "LCSC Part #" "C17855"
 			(at 170.18 151.13 0)
 			(show_name no)
@@
 			)
 		)
-		(property "Value" "EMERALD"
+		(property "Value" "ORANGE/0603"
 			(at 73.66 118.11 90)
 			(show_name no)
@@
 			)
 		)
-		(property "Mfr PN" "19-213/GHC-XS1T1N/5T"
+		(property "Mfr PN" "19-217/S2C-AL1M2VY/6T"
 			(at 76.2 118.11 0)
 			(hide yes)
@@
 			)
 		)
-		(property "Vendor PN" "C2984266"
+		(property "Vendor PN" "C2987557"
 			(at 76.2 118.11 0)
 			(hide yes)
@@
 			)
 		)
-		(property "LCSC Part #" "C2984266"
+		(property "LCSC Part #" "C2987557"
 			(at 73.66 120.65 90)
 			(show_name no)
@@
 			)
 		)
-		(property "Value" "10k/125mW"
+		(property "Value" "9.1k/125mW"
 			(at 73.66 31.75 0)
 			(show_name no)
@@
 			)
 		)
-		(property "Mfr PN" "0805W8F1002T5E"
+		(property "Mfr PN" "0805W8F9101T5E"
 			(at 76.2 31.75 0)
 			(hide yes)
@@
 			)
 		)
-		(property "Vendor PN" "C17414"
+		(property "Vendor PN" "C17855"
 			(at 76.2 31.75 0)
 			(hide yes)
@@
 			)
 		)
-		(property "LCSC Part #" "C17414"
+		(property "LCSC Part #" "C17855"
 			(at 73.66 34.29 0)
 			(show_name no)
@@
 			)
 		)
-		(property "Value" "10k/125mW"
+		(property "Value" "9.1k/125mW"
 			(at 73.66 107.95 0)
 			(show_name no)
@@
 			)
 		)
-		(property "Mfr PN" "0805W8F1002T5E"
+		(property "Mfr PN" "0805W8F9101T5E"
 			(at 76.2 107.95 0)
 			(hide yes)
@@
 			)
 		)
-		(property "Vendor PN" "C17414"
+		(property "Vendor PN" "C17855"
 			(at 76.2 107.95 0)
 			(hide yes)
@@
 			)
 		)
-		(property "LCSC Part #" "C17414"
+		(property "LCSC Part #" "C17855"
 			(at 73.66 110.49 0)
 			(show_name no)
@@
 			)
 		)
-		(property "Value" "EMERALD"
+		(property "Value" "ORANGE/0603"
 			(at 73.66 80.01 90)
 			(show_name no)
@@
 			)
 		)
-		(property "Mfr PN" "19-213/GHC-XS1T1N/5T"
+		(property "Mfr PN" "19-217/S2C-AL1M2VY/6T"
 			(at 76.2 80.01 0)
 			(hide yes)
@@
 			)
 		)
-		(property "Vendor PN" "C2984266"
+		(property "Vendor PN" "C2987557"
 			(at 76.2 80.01 0)
 			(hide yes)
@@
 			)
 		)
-		(property "LCSC Part #" "C2984266"
+		(property "LCSC Part #" "C2987557"
 			(at 73.66 82.55 90)
 			(show_name no)
@@
 			)
 		)
-		(property "Value" "10k/125mW"
+		(property "Value" "9.1k/125mW"
 			(at 73.66 69.85 0)
 			(show_name no)
@@
 			)
 		)
-		(property "Mfr PN" "0805W8F1002T5E"
+		(property "Mfr PN" "0805W8F9101T5E"
 			(at 76.2 69.85 0)
 			(hide yes)
@@
 			)
 		)
-		(property "Vendor PN" "C17414"
+		(property "Vendor PN" "C17855"
 			(at 76.2 69.85 0)
 			(hide yes)
@@
 			)
 		)
-		(property "LCSC Part #" "C17414"
+		(property "LCSC Part #" "C17855"
 			(at 73.66 72.39 0)
 			(show_name no)
@@
 			)
 		)
-		(property "Value" "EMERALD"
+		(property "Value" "ORANGE/0603"
 			(at 170.18 158.75 90)
 			(show_name no)
@@
 			)
 		)
-		(property "Mfr PN" "19-213/GHC-XS1T1N/5T"
+		(property "Mfr PN" "19-217/S2C-AL1M2VY/6T"
 			(at 172.72 158.75 0)
 			(hide yes)
@@
 			)
 		)
-		(property "Vendor PN" "C2984266"
+		(property "Vendor PN" "C2987557"
 			(at 172.72 158.75 0)
 			(hide yes)
@@
 			)
 		)
-		(property "LCSC Part #" "C2984266"
+		(property "LCSC Part #" "C2987557"
 			(at 170.18 161.29 90)
 			(show_name no)
@@
 			)
 		)
-		(property "Value" "10k/125mW"
+		(property "Value" "9.1k/125mW"
 			(at 170.18 72.39 0)
 			(show_name no)
@@
 			)
 		)
-		(property "Mfr PN" "0805W8F1002T5E"
+		(property "Mfr PN" "0805W8F9101T5E"
 			(at 172.72 72.39 0)
 			(hide yes)
@@
 			)
 		)
-		(property "Vendor PN" "C17414"
+		(property "Vendor PN" "C17855"
 			(at 172.72 72.39 0)
 			(hide yes)
@@
 			)
 		)
-		(property "LCSC Part #" "C17414"
+		(property "LCSC Part #" "C17855"
 			(at 170.18 74.93 0)
 			(show_name no)
@@
 			)
 		)
-		(property "Value" "EMERALD"
+		(property "Value" "ORANGE/0603"
 			(at 73.66 41.91 90)
 			(show_name no)
@@
 			)
 		)
-		(property "Mfr PN" "19-213/GHC-XS1T1N/5T"
+		(property "Mfr PN" "19-217/S2C-AL1M2VY/6T"
 			(at 76.2 41.91 0)
 			(hide yes)
@@
 			)
 		)
-		(property "Vendor PN" "C2984266"
+		(property "Vendor PN" "C2987557"
 			(at 76.2 41.91 0)
 			(hide yes)
@@
 			)
 		)
-		(property "LCSC Part #" "C2984266"
+		(property "LCSC Part #" "C2987557"
 			(at 73.66 44.45 90)
 			(show_name no)
@@
 			)
 		)
-		(property "Value" "10k/125mW"
+		(property "Value" "9.1k/125mW"
 			(at 73.66 146.05 0)
 			(show_name no)
@@
 			)
 		)
-		(property "Mfr PN" "0805W8F1002T5E"
+		(property "Mfr PN" "0805W8F9101T5E"
 			(at 76.2 146.05 0)
 			(hide yes)
@@
 			)
 		)
-		(property "Vendor PN" "C17414"
+		(property "Vendor PN" "C17855"
 			(at 76.2 146.05 0)
 			(hide yes)
@@
 			)
 		)
-		(property "LCSC Part #" "C17414"
+		(property "LCSC Part #" "C17855"
 			(at 73.66 148.59 0)
 			(show_name no)
@@
 			)
 		)
-		(property "Value" "10k/125mW"
+		(property "Value" "9.1k/125mW"
 			(at 170.18 34.29 0)
 			(show_name no)
@@
 			)
 		)
-		(property "Mfr PN" "0805W8F1002T5E"
+		(property "Mfr PN" "0805W8F9101T5E"
 			(at 172.72 34.29 0)
 			(hide yes)
@@
 			)
 		)
-		(property "Vendor PN" "C17414"
+		(property "Vendor PN" "C17855"
 			(at 172.72 34.29 0)
 			(hide yes)
@@
 			)
 		)
-		(property "LCSC Part #" "C17414"
+		(property "LCSC Part #" "C17855"
 			(at 170.18 36.83 0)
 			(show_name no)
@@
 			)
 		)
-		(property "Value" "EMERALD"
+		(property "Value" "ORANGE/0603"
 			(at 170.18 120.65 90)
 			(show_name no)
@@
 			)
 		)
-		(property "Mfr PN" "19-213/GHC-XS1T1N/5T"
+		(property "Mfr PN" "19-217/S2C-AL1M2VY/6T"
 			(at 172.72 120.65 0)
 			(hide yes)
@@
 			)
 		)
-		(property "Vendor PN" "C2984266"
+		(property "Vendor PN" "C2987557"
 			(at 172.72 120.65 0)
 			(hide yes)
@@
 			)
 		)
-		(property "LCSC Part #" "C2984266"
+		(property "LCSC Part #" "C2987557"
 			(at 170.18 123.19 90)
 			(show_name no)
@@
 			)
 		)
-		(property "Value" "EMERALD"
+		(property "Value" "ORANGE/0603"
 			(at 170.18 44.45 90)
 			(show_name no)
@@
 			)
 		)
-		(property "Mfr PN" "19-213/GHC-XS1T1N/5T"
+		(property "Mfr PN" "19-217/S2C-AL1M2VY/6T"
 			(at 172.72 44.45 0)
 			(hide yes)
@@
 			)
 		)
-		(property "Vendor PN" "C2984266"
+		(property "Vendor PN" "C2987557"
 			(at 172.72 44.45 0)
 			(hide yes)
@@
 			)
 		)
-		(property "LCSC Part #" "C2984266"
+		(property "LCSC Part #" "C2987557"
 			(at 170.18 46.99 90)
 			(show_name no)

Commit message: LEDs replaced for orange
Parts:
- R1, R2, R3, R4, R5, R6, R7, R8: value 9.1k/125mW -> 10k/125mW; LCSC Part # C17855 -> C17414; Mfr PN 0805W8F9101T5E -> 0805W8F1002T5E; Vendor PN C17855 -> C17414
Other:
- note added: "V_{F} = 1,8V @ 2,5mA I_{LED} = (24V - V_{F}) / R I_{LED} = (24V - 1.8V) / 10k I_{LED} = 2.22 mA"
- note removed: "V_{F} = 1,8V @ 2,5mA I_{LED} = (24V - V_{F}) / R I_{LED} = (24V - 1.8V) / 9.1k I_{LED} = 2.44 mA"
Changed lines of the file:
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@@
 		(rev "V1.2")
 	)
-	(text "V_{F} = 1,8V @ 2,5mA\nI_{LED} = (24V - V_{F}) / R\nI_{LED} = (24V - 1.8V) / 9.1k\nI_{LED} = 2.44 mA"
+	(text "V_{F} = 1,8V @ 2,5mA\nI_{LED} = (24V - V_{F}) / R\nI_{LED} = (24V - 1.8V) / 10k\nI_{LED} = 2.22 mA"
 		(exclude_from_sim no)
 		(at 66.04 179.07 0)
@@
 			)
 		)
-		(property "Value" "9.1k/125mW"
+		(property "Value" "10k/125mW"
 			(at 170.18 110.49 0)
 			(show_name no)
@@
 			)
 		)
-		(property "Mfr PN" "0805W8F9101T5E"
+		(property "Mfr PN" "0805W8F1002T5E"
 			(at 172.72 110.49 0)
 			(hide yes)
@@
 			)
 		)
-		(property "Vendor PN" "C17855"
+		(property "Vendor PN" "C17414"
 			(at 172.72 110.49 0)
 			(hide yes)
@@
 			)
 		)
-		(property "LCSC Part #" "C17855"
+		(property "LCSC Part #" "C17414"
 			(at 170.18 113.03 0)
 			(show_name no)
@@
 			)
 		)
-		(property "Value" "9.1k/125mW"
+		(property "Value" "10k/125mW"
 			(at 170.18 148.59 0)
 			(show_name no)
@@
 			)
 		)
-		(property "Mfr PN" "0805W8F9101T5E"
+		(property "Mfr PN" "0805W8F1002T5E"
 			(at 172.72 148.59 0)
 			(hide yes)
@@
 			)
 		)
-		(property "Vendor PN" "C17855"
+		(property "Vendor PN" "C17414"
 			(at 172.72 148.59 0)
 			(hide yes)
@@
 			)
 		)
-		(property "LCSC Part #" "C17855"
+		(property "LCSC Part #" "C17414"
 			(at 170.18 151.13 0)
 			(show_name no)
@@
 			)
 		)
-		(property "Value" "9.1k/125mW"
+		(property "Value" "10k/125mW"
 			(at 73.66 31.75 0)
 			(show_name no)
@@
 			)
 		)
-		(property "Mfr PN" "0805W8F9101T5E"
+		(property "Mfr PN" "0805W8F1002T5E"
 			(at 76.2 31.75 0)
 			(hide yes)
@@
 			)
 		)
-		(property "Vendor PN" "C17855"
+		(property "Vendor PN" "C17414"
 			(at 76.2 31.75 0)
 			(hide yes)
@@
 			)
 		)
-		(property "LCSC Part #" "C17855"
+		(property "LCSC Part #" "C17414"
 			(at 73.66 34.29 0)
 			(show_name no)
@@
 			)
 		)
-		(property "Value" "9.1k/125mW"
+		(property "Value" "10k/125mW"
 			(at 73.66 107.95 0)
 			(show_name no)
@@
 			)
 		)
-		(property "Mfr PN" "0805W8F9101T5E"
+		(property "Mfr PN" "0805W8F1002T5E"
 			(at 76.2 107.95 0)
 			(hide yes)
@@
 			)
 		)
-		(property "Vendor PN" "C17855"
+		(property "Vendor PN" "C17414"
 			(at 76.2 107.95 0)
 			(hide yes)
@@
 			)
 		)
-		(property "LCSC Part #" "C17855"
+		(property "LCSC Part #" "C17414"
 			(at 73.66 110.49 0)
 			(show_name no)
@@
 			)
 		)
-		(property "Value" "9.1k/125mW"
+		(property "Value" "10k/125mW"
 			(at 73.66 69.85 0)
 			(show_name no)
@@
 			)
 		)
-		(property "Mfr PN" "0805W8F9101T5E"
+		(property "Mfr PN" "0805W8F1002T5E"
 			(at 76.2 69.85 0)
 			(hide yes)
@@
 			)
 		)
-		(property "Vendor PN" "C17855"
+		(property "Vendor PN" "C17414"
 			(at 76.2 69.85 0)
 			(hide yes)
@@
 			)
 		)
-		(property "LCSC Part #" "C17855"
+		(property "LCSC Part #" "C17414"
 			(at 73.66 72.39 0)
 			(show_name no)
@@
 			)
 		)
-		(property "Value" "9.1k/125mW"
+		(property "Value" "10k/125mW"
 			(at 170.18 72.39 0)
 			(show_name no)
@@
 			)
 		)
-		(property "Mfr PN" "0805W8F9101T5E"
+		(property "Mfr PN" "0805W8F1002T5E"
 			(at 172.72 72.39 0)
 			(hide yes)
@@
 			)
 		)
-		(property "Vendor PN" "C17855"
+		(property "Vendor PN" "C17414"
 			(at 172.72 72.39 0)
 			(hide yes)
@@
 			)
 		)
-		(property "LCSC Part #" "C17855"
+		(property "LCSC Part #" "C17414"
 			(at 170.18 74.93 0)
 			(show_name no)
@@
 			)
 		)
-		(property "Value" "9.1k/125mW"
+		(property "Value" "10k/125mW"
 			(at 73.66 146.05 0)
 			(show_name no)
@@
 			)
 		)
-		(property "Mfr PN" "0805W8F9101T5E"
+		(property "Mfr PN" "0805W8F1002T5E"
 			(at 76.2 146.05 0)
 			(hide yes)
@@
 			)
 		)
-		(property "Vendor PN" "C17855"
+		(property "Vendor PN" "C17414"
 			(at 76.2 146.05 0)
 			(hide yes)
@@
 			)
 		)
-		(property "LCSC Part #" "C17855"
+		(property "LCSC Part #" "C17414"
 			(at 73.66 148.59 0)
 			(show_name no)
@@
 			)
 		)
-		(property "Value" "9.1k/125mW"
+		(property "Value" "10k/125mW"
 			(at 170.18 34.29 0)
 			(show_name no)
@@
 			)
 		)
-		(property "Mfr PN" "0805W8F9101T5E"
+		(property "Mfr PN" "0805W8F1002T5E"
 			(at 172.72 34.29 0)
 			(hide yes)
@@
 			)
 		)
-		(property "Vendor PN" "C17855"
+		(property "Vendor PN" "C17414"
 			(at 172.72 34.29 0)
 			(hide yes)
@@
 			)
 		)
-		(property "LCSC Part #" "C17855"
+		(property "LCSC Part #" "C17414"
 			(at 170.18 36.83 0)
 			(show_name no)

Commit message: Adjusted component rotation and offset information for JLCPCB.
Parts:
- D1, D11, D13, D15, D3, D5, D7, D9: Case (none) -> 0603/1608; JLCPCB BOM 1 -> (none); Package 0603/1608 -> (none)
- D10, D12, D14, D16, D2, D4, D6, D8: Case (none) -> SOD-123; JLCPCB BOM 1 -> (none); Package SOD-123 -> (none)
- J1, J2, J3, K1, K2, K3, K4, K5, K6, K7, K8: JLCPCB BOM 1 -> (none)
- J4, J5, J6, J7: FT Rotation Offset (none) -> 180; JLCPCB BOM 1 -> (none)
- R1, R2, R3, R4, R5, R6, R7, R8: Case (none) -> 0805/2012; JLCPCB BOM 1 -> (none); Package 0805/2012 -> (none)
- RV1, RV2, RV3, RV4, RV5, RV6, RV7, RV8: Case (none) -> 9.5x5.08mm; JLCPCB BOM 1 -> (none); Package 9.5x5.08mm -> (none); Technology MOV -> (none)
