File: V1/eumesmo-rl-8ch8a-v1.kicad_sch (KiCad schematic)
At the start: 47 parts, among them J1 250-202, J2 250-204, J3 250-204, J4 DB142V-5.08-4P, J5 DB142V-5.08-4P, J6 DB142V-5.08-4P, J7 DB142V-5.08-4P, K1 G5Q-1A4-DC24V, K2 G5Q-1A4-DC24V, K3 G5Q-1A4-DC24V, K4 G5Q-1A4-DC24V, K5 G5Q-1A4-DC24V, K6 G5Q-1A4-DC24V, K7 G5Q-1A4-DC24V, K8 G5Q-1A4-DC24V

Commit message: Replaced Wago connectors for other brand, no stock.
Parts:
- J1: LCSC Part # C2765061 -> C475154; Mfr Wago -> Cixi Kefa Elec; Mfr PN 250-202 -> KF250-3.5-2P-1; Vendor PN C2765061 -> C475154
- J2, J3: LCSC Part # C2765063 -> C475156; Mfr Wago -> Cixi Kefa Elec; Mfr PN 250-204 -> KF250-3.5-4P-1; Vendor PN C2765063 -> C475156
Changed lines of the file:
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@@
 			)
 		)
-		(property "LCSC Part #" "C2765063"
+		(property "LCSC Part #" "C475156"
 			(at 35.56 128.27 0)
 			(hide yes)
@@
 			)
 		)
-		(property "Mfr" "Wago"
+		(property "Mfr" "Cixi Kefa Elec"
 			(at 35.56 128.27 0)
 			(hide yes)
@@
 			)
 		)
-		(property "Mfr PN" "250-204"
+		(property "Mfr PN" "KF250-3.5-4P-1"
 			(at 35.56 128.27 0)
 			(hide yes)
@@
 			)
 		)
-		(property "Vendor PN" "C2765063"
+		(property "Vendor PN" "C475156"
 			(at 35.56 128.27 0)
 			(hide yes)
@@
 			)
 		)
-		(property "LCSC Part #" "C2765061"
+		(property "LCSC Part #" "C475154"
 			(at 35.56 35.56 0)
 			(hide yes)
@@
 			)
 		)
-		(property "Mfr" "Wago"
+		(property "Mfr" "Cixi Kefa Elec"
 			(at 35.56 35.56 0)
 			(hide yes)
@@
 			)
 		)
-		(property "Mfr PN" "250-202"
+		(property "Mfr PN" "KF250-3.5-2P-1"
 			(at 35.56 35.56 0)
 			(hide yes)
@@
 			)
 		)
-		(property "Vendor PN" "C2765061"
+		(property "Vendor PN" "C475154"
 			(at 35.56 35.56 0)
 			(hide yes)
@@
 			)
 		)
-		(property "LCSC Part #" "C2765063"
+		(property "LCSC Part #" "C475156"
 			(at 35.56 52.07 0)
 			(hide yes)
@@
 			)
 		)
-		(property "Mfr" "Wago"
+		(property "Mfr" "Cixi Kefa Elec"
 			(at 35.56 52.07 0)
 			(hide yes)
@@
 			)
 		)
-		(property "Mfr PN" "250-204"
+		(property "Mfr PN" "KF250-3.5-4P-1"
 			(at 35.56 52.07 0)
 			(hide yes)
@@
 			)
 		)
-		(property "Vendor PN" "C2765063"
+		(property "Vendor PN" "C475156"
 			(at 35.56 52.07 0)
 			(hide yes)
